File: esp32-prog.kicad_sch (KiCad schematic)
At the start: 43 parts, among them J1 USB_B_Micro_10118194-0001LF, J2 1.27mm_50mils_male_DW127R-22-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, Q1 AO3400A, Q2 AO3400A, SW1 SW_DIP_x02_50mil_1.27mm_TP-02, U1 AMS1117-3.3, U2 SRV05-4, U3 CH340C, U4 74LVC1G125GW_Nexperia, U5 74LVC1G125GW_Nexperia, U6 74LVC1G125GW_Nexperia, U7 74LVC1G125GW_Nexperia

Commit message: fab: fix 4.7u cap and buffer FP
Parts:
- C2, C3, C5: value 22u_1206_CL31A226KPHNNNE -> 4.7u_1206_1206B475K500NT; symbol 00-kiml-capacitors-smd:22u_1206_CL31A226KPHNNNE -> 00-kiml-capacitors-smd:4.7u_1206_1206B475K500NT; LNK1 https://jlcpcb.com/partdetail/6131-CL31A226KPHNNNE/C5672 -> https://jlcpcb.com/partdetail/30577-1206B475K500NT/C29823; MFR Samsung -> FH; MPN CL31A226KPHNNNE -> 1206B475K500NT; Rating 10V -> 50V; SPN1 C5672 -> C29823; UserValue 22u -> 4.7u
- U4, U5, U6, U7: footprint Package_TO_SOT_SMD:SOT-23-5 -> Package_TO_SOT_SMD:SOT-353_SC-70-5
Connections:
- net +5V: no longer C5.1, C6.1
- net VBUS: now also C5.1, C6.1
